File: sed1200emu.kicad_pcb (KiCad board)
At the start: 2 copper layers, 46.2 x 38.9 mm, 17 parts, among them CN1 PINHD-1X6, CN2 PINHD-1X6, IC1 MEGA8-AI, Q1 CRYSTALHC49S

Commit message: Fix more Rule Violations
Parts:
- moved SCK1 1.50 mm to (154.0, 106.0)
- moved MISO1 0.95 mm to (153.7, 110.5)
Routing:
- net Net-(IC1-PB4(MISO)): track 6.20 -> 4.97 mm
- net Net-(IC1-PB5(SCK)): track 3.78 -> 4.99 mm
Changed lines of the file:
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@@
   )
   (footprint "Connector_PinHeader_2.54mm:PinHeader_1x01_P2.54mm_Vertical" (layer "F.Cu")
-    (at 154 107.5)
+    (at 154 106)
     (descr "Through hole straight pin header, 1x01, 2.54mm pitch, single row")
     (tags "Through hole pin header THT 1x01 2.54mm single row")
@@
   )
   (footprint "Connector_PinHeader_2.54mm:PinHeader_1x01_P2.54mm_Vertical" (layer "F.Cu")
-    (at 153.663904 111.451628)
+    (at 153.663904 110.5)
     (descr "Through hole straight pin header, 1x01, 2.54mm pitch, single row")
     (tags "Through hole pin header THT 1x01 2.54mm single row")
@@
   (segment (start 140.5951 106.5796) (end 142.0031 106.5796) (width 0.3) (layer "F.Cu") (net 2))
   (segment (start 129.747634 97.501066) (end 129.804566 97.501066) (width 0.3) (layer "F.Cu") (net 2))
-  (segment (start 129.747634 91.752366) (end 129.5 92) (width 0.3) (layer "F.Cu") (net 2))
   (segment (start 169.6211 104.5516) (end 169.6211 120.1116) (width 0.3) (layer "F.Cu") (net 2))
   (segment (start 158.2571 122.9056) (end 158.1911 122.8396) (width 0.3) (layer "F.Cu") (net 2))
@@
   (segment (start 147.4531 106.5796) (end 148.2531 107.3796) (width 0.3) (layer "F.Cu") (net 2))
   (segment (start 158.1911 122.8396) (end 130.6931 122.8396) (width 0.3) (layer "F.Cu") (net 2))
-  (segment (start 133.3651 101.0616) (end 133.308168 101.0616) (width 0.3) (layer "F.Cu") (net 2))
   (segment (start 169.6211 120.1116) (end 166.8271 122.9056) (width 0.3) (layer "F.Cu") (net 2))
   (segment (start 148.2531 107.3796) (end 150.5031 107.3796) (width 0.3) (layer "F.Cu") (net 2))
@@
   (segment (start 154.570831 114.333869) (end 156.6671 112.2376) (width 0.2) (layer "F.Cu") (net 25))
   (segment (start 151.705265 114.333869) (end 154.570831 114.333869) (width 0.2) (layer "F.Cu") (net 25))
-  (segment (start 149.0531 111.0531) (end 149.0531 109.6296) (width 0.2) (layer "F.Cu") (net 28))
-  (segment (start 149.451628 111.451628) (end 149.0531 111.0531) (width 0.2) (layer "F.Cu") (net 28))
-  (segment (start 153.663904 111.451628) (end 149.451628 111.451628) (width 0.2) (layer "F.Cu") (net 28))
-  (segment (start 154 107.5) (end 153.3204 108.1796) (width 0.2) (layer "F.Cu") (net 29))
-  (segment (start 153.3204 108.1796) (end 150.5031 108.1796) (width 0.2) (layer "F.Cu") (net 29))
+  (segment (start 149.0531 109.6296) (end 152.793504 109.6296) (width 0.2) (layer "F.Cu") (net 28))
+  (segment (start 152.793504 109.6296) (end 153.663904 110.5) (width 0.2) (layer "F.Cu") (net 28))
+  (segment (start 152.8204 108.1796) (end 154 107) (width 0.2) (layer "F.Cu") (net 29))
+  (segment (start 150.5031 108.1796) (end 152.8204 108.1796) (width 0.2) (layer "F.Cu") (net 29))
+  (segment (start 154 107) (end 154 106) (width 0.2) (layer "F.Cu") (net 29))
   (segment (start 145.8531 97.8531) (end 145 97) (width 0.2) (layer "F.Cu") (net 34))
   (segment (start 145.8531 101.1296) (end 145.8531 97.8531) (width 0.2) (layer "F.Cu") (net 34))
